File: final.brd (EAGLE design)
At the start: 107.9 x 75.2 mm, 32 parts, among them IC1 LM741P, IC2 LM741P, IC3 LM741D, IC4 LM741P, IC5 LM741P

Commit message: choHo_2
Parts:
- moved R8 18.1 mm to (84.5, 59.1)
Changed lines of the file:
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@@
 <element name="POWER1" library="pinhead" package="1X02" value="" x="19.685" y="63.5"/>
 <element name="POWER2" library="pinhead" package="1X02" value="" x="29.845" y="63.5"/>
-<element name="R8" library="resistor" package="R0805" value="32k" x="66.675" y="62.23" rot="R90"/>
+<element name="R8" library="resistor" package="R0805" value="32k" x="84.455" y="59.055" rot="R90"/>
 <element name="R9" library="resistor" package="R0805" value="32k" x="73.66" y="62.23" rot="R90"/>
 <element name="R11" library="resistor" package="R0805" value="32k" x="52.07" y="57.15"/>
@@
 <contactref element="R8" pad="2"/>
 <contactref element="R9" pad="2"/>
-<wire x1="66.675" y1="63.08" x2="73.66" y2="63.08" width="0" layer="19" extent="1-1"/>
-<wire x1="31.115" y1="63.5" x2="66.675" y2="63.08" width="0" layer="19" extent="1-1"/>
+<wire x1="84.455" y1="59.905" x2="73.66" y2="63.08" width="0" layer="19" extent="1-1"/>
+<wire x1="31.115" y1="63.5" x2="84.455" y2="59.905" width="0" layer="19" extent="1-1"/>
 </signal>
 <signal name="N$11">
@@
 <contactref element="IC4" pad="5"/>
 <contactref element="TEMP_IN" pad="2"/>
-<wire x1="66.675" y1="55.88" x2="66.675" y2="61.38" width="0" layer="19" extent="1-1"/>
-<wire x1="59.055" y1="63.5" x2="66.675" y2="61.38" width="0" layer="19" extent="1-1"/>
+<wire x1="66.675" y1="55.88" x2="84.455" y2="58.205" width="0" layer="19" extent="1-1"/>
+<wire x1="59.055" y1="63.5" x2="84.455" y2="58.205" width="0" layer="19" extent="1-1"/>
 </signal>
 <signal name="N$12">
